File: A1000_RAM_Expansion_extended.kicad_pcb (KiCad board)
At the start: 2 copper layers, 149.5 x 51.5 mm, 37 parts, among them J1 Front_Connector, J2 Conn_02x05, U1 XC9572XL-xxVQx64, U2 LD1117S33TR_SOT223

Commit message: PCB Cleanup
Other:
- board size 149.5 x 51.5 mm -> 149.5 x 51.6 mm
