File: A1000_RAM_Expansion_extended.kicad_sch (KiCad schematic)
At the start: 24 parts, among them J1 Front_Connector, J2 Conn_02x05_Odd_Even, U1 XC9572XL-xxVQx64, U2 LD1117S33TR_SOT223

Commit message: Cleanup
Connections:
- net D0: now also J1.16 (Pin_16); no longer J1.T (Pin_46)
- net D1: now also J1.T (Pin_46); no longer J1.16 (Pin_16)
- net D10: now also J1.F (Pin_36); no longer J1.6 (Pin_6)
- net D11: now also J1.6 (Pin_6); no longer J1.F (Pin_36)
- net D12: now also J1.4 (Pin_4); no longer J1.D (Pin_34)
- net D13: now also J1.D (Pin_34); no longer J1.4 (Pin_4)
- net D14: now also J1.B (Pin_32); no longer J1.2 (Pin_2)
- net D15: now also J1.2 (Pin_2); no longer J1.B (Pin_32)
- net D2: now also J1.R (Pin_44); no longer J1.14 (Pin_14)
- net D3: now also J1.14 (Pin_14); no longer J1.R (Pin_44)
- net D4: now also J1.12 (Pin_12); no longer J1.N (Pin_42)
- net D5: now also J1.N (Pin_42); no longer J1.12 (Pin_12)
- net D6: now also J1.L (Pin_40); no longer J1.10 (Pin_10)
- net D7: now also J1.10 (Pin_10); no longer J1.L (Pin_40)
- net D8: now also J1.8 (Pin_8); no longer J1.J (Pin_38)
- net D9: now also J1.J (Pin_38); no longer J1.8 (Pin_8)
- net DRA0: now also J1.Y (Pin_51); no longer J1.21 (Pin_21)
- net DRA1: now also J1.X (Pin_50); no longer J1.20 (Pin_20)
- net DRA2: now also J1.W (Pin_49); no longer J1.19 (Pin_19)
- net DRA3: now also J1.V (Pin_48); no longer J1.18 (Pin_18)
- net DRA4: now also J1.18 (Pin_18); no longer J1.V (Pin_48)
- net DRA5: now also J1.19 (Pin_19); no longer J1.W (Pin_49)
- net DRA6: now also J1.20 (Pin_20); no longer J1.X (Pin_50)
- net DRA7: now also J1.21 (Pin_21); no longer J1.Y (Pin_51)
- net GND: now also SRAM_2.24 (GND)
- net /CASL0: now also J1.28 (Pin_28); no longer J1.FF (Pin_58)
- net /CASL1: now also J1.FF (Pin_58); no longer J1.28 (Pin_28)
- net /CASU0: now also J1.26 (Pin_26); no longer J1.DD (Pin_56)
- net /CASU1: now also J1.DD (Pin_56); no longer J1.26 (Pin_26)
- net /RAS: now also J1.23 (Pin_23); no longer J1.AA (Pin_53)
- net /RRW: now also J1.AA (Pin_53); no longer J1.23 (Pin_23)
- no-connect marks 0 -> 16
Other:
- moved on the sheet: RN4
