File: _autosave-A1000_RAM_Expansion_extended.kicad_pcb (KiCad board)
At the start: 2 copper layers, 149.5 x 51.6 mm, 37 parts, among them J1 Front_Connector, J2 Conn_02x05, U1 XC9572XL-xxVQx64, U2 LD1117S33TR_SOT223

Commit message: Cleanup
Parts:
- J2: value Conn_02x05 -> Conn_02x05_Odd_Even
Changed lines of the file:
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@@
 			)
 		)
-		(property "Value" "Conn_02x05"
+		(property "Value" "Conn_02x05_Odd_Even"
 			(at 1.125 -6.795 90)
 			(layer "F.Fab")
@@
 			(net 48 "unconnected-(U1-I{slash}O-Pad1)")
 			(pinfunction "I/O")
-			(pintype "bidirectional")
+			(pintype "bidirectional+no_connect")
 		)
 		(pad "2" smd roundrect
@@
 			(net 55 "unconnected-(U1-I{slash}O{slash}GTS2-Pad2)")
 			(pinfunction "I/O/GTS2")
-			(pintype "bidirectional")
+			(pintype "bidirectional+no_connect")
 		)
 		(pad "3" smd roundrect
@@
 			(net 57 "unconnected-(U1-I{slash}O-Pad4)")
 			(pinfunction "I/O")
-			(pintype "bidirectional")
+			(pintype "bidirectional+no_connect")
 		)
 		(pad "5" smd roundrect
@@
 			(net 62 "unconnected-(U1-I{slash}O{slash}GTS1-Pad5)")
 			(pinfunction "I/O/GTS1")
-			(pintype "bidirectional")
+			(pintype "bidirectional+no_connect")
 		)
 		(pad "6" smd roundrect
@@
 			(net 71 "unconnected-(U1-I{slash}O-Pad7)")
 			(pinfunction "I/O")
-			(pintype "bidirectional")
+			(pintype "bidirectional+no_connect")
 		)
 		(pad "8" smd roundrect
@@
 			(net 61 "unconnected-(U1-I{slash}O{slash}GCK2-Pad16)")
 			(pinfunction "I/O/GCK2")
-			(pintype "bidirectional")
+			(pintype "bidirectional+no_connect")
 		)
 		(pad "17" smd roundrect
@@
 			(net 56 "unconnected-(U1-I{slash}O{slash}GCK3-Pad17)")
 			(pinfunction "I/O/GCK3")
-			(pintype "bidirectional")
+			(pintype "bidirectional+no_connect")
 		)
 		(pad "18" smd roundrect
@@
 			(net 70 "unconnected-(U1-I{slash}O-Pad19)")
 			(pinfunction "I/O")
-			(pintype "bidirectional")
+			(pintype "bidirectional+no_connect")
 		)
 		(pad "20" smd roundrect
@@
 			(net 68 "unconnected-(U1-I{slash}O-Pad23)")
 			(pinfunction "I/O")
-			(pintype "bidirectional")
+			(pintype "bidirectional+no_connect")
 		)
 		(pad "24" smd roundrect
@@
 			(net 50 "unconnected-(U1-I{slash}O-Pad43)")
 			(pinfunction "I/O")
-			(pintype "bidirectional")
+			(pintype "bidirectional+no_connect")
 		)
 		(pad "44" smd roundrect
@@
 			(net 60 "unconnected-(U1-I{slash}O-Pad46)")
 			(pinfunction "I/O")
-			(pintype "bidirectional")
+			(pintype "bidirectional+no_connect")
 		)
 		(pad "47" smd roundrect
@@
 			(net 59 "unconnected-(U1-I{slash}O-Pad52)")
 			(pinfunction "I/O")
-			(pintype "bidirectional")
+			(pintype "bidirectional+no_connect")
 		)
 		(pad "53" smd roundrect
@@
 			(net 49 "unconnected-(U1-I{slash}O-Pad61)")
 			(pinfunction "I/O")
-			(pintype "bidirectional")
+			(pintype "bidirectional+no_connect")
 		)
 		(pad "62" smd roundrect
@@
 			(net 65 "unconnected-(U1-I{slash}O-Pad62)")
 			(pinfunction "I/O")
-			(pintype "bidirectional")
+			(pintype "bidirectional+no_connect")
 		)
 		(pad "63" smd roundrect
@@
 			(net 72 "unconnected-(U1-I{slash}O-Pad63)")
 			(pinfunction "I/O")
-			(pintype "bidirectional")
+			(pintype "bidirectional+no_connect")
 		)
 		(pad "64" smd roundrect
@@
 			(net 58 "unconnected-(U1-I{slash}O{slash}GSR-Pad64)")
 			(pinfunction "I/O/GSR")
-			(pintype "bidirectional")
+			(pintype "bidirectional+no_connect")
 		)
 		(embedded_fonts no)
@@
 	)
 	(zone
+		(net 73)
+		(net_name "GND")
+		(layer "F.Cu")
+		(hatch edge 0.5)
+		(priority 1)
+		(connect_pads
+			(clearance 0.5)
+		)
+		(min_thickness 0.25)
+		(filled_areas_thickness no)
+		(fill yes
+			(thermal_gap 0.5)
+			(thermal_bridge_width 0.5)
+		)
+		(polygon
+			(pts
+				(xy 70.584623 56.5) (xy 220.959623 56.5) (xy 221.115384 108.994132) (xy 70.740384 108.869132)
+			)
+		)
+	)
+	(zone
 		(net 1)
 		(net_name "+3.3V")
@@
 		(net 73)
 		(net_name "GND")
-		(layer "F.Cu")
-		(hatch edge 0.5)
-		(priority 1)
-		(connect_pads
-			(clearance 0.5)
-		)
-		(min_thickness 0.25)
-		(filled_areas_thickness no)
-		(fill yes
-			(thermal_gap 0.5)
-			(thermal_bridge_width 0.5)
-		)
-		(polygon
-			(pts
-				(xy 70.584623 56.5) (xy 220.959623 56.5) (xy 221.115384 108.994132) (xy 70.740384 108.869132)
-			)
-		)
-	)
-	(zone
-		(net 73)
-		(net_name "GND")
 		(layer "B.Cu")
 		(hatch edge 0.5)
@@
 		(name "$teardrop_padvia$")
 		(hatch none 0.1)
-		(priority 30000)
+		(priority 30001)
 		(attr
 			(teardrop
@@
 		(polygon
 			(pts
-				(xy 96.721964 74.381589) (xy 96.368411 74.028036) (xy 95.958329 74.375559) (xy 96.124293 74.625707)
-				(xy 96.374441 74.791671)
+				(xy 95.530764 74.525) (xy 95.530764 74.725) (xy 96.066473 74.919236) (xy 96.126 74.625) (xy 96.066473 74.330764)
 			)
 		)
@@
 		(name "$teardrop_padvia$")
 		(hatch none 0.1)
-		(priority 30001)
+		(priority 30000)
 		(attr
 			(teardrop
@@
 		(polygon
 			(pts
-				(xy 95.530764 74.525) (xy 95.530764 74.725) (xy 96.066473 74.919236) (xy 96.126 74.625) (xy 96.066473 74.330764)
+				(xy 96.721964 74.381589) (xy 96.368411 74.028036) (xy 95.958329 74.375559) (xy 96.124293 74.625707)
+				(xy 96.374441 74.791671)
 			)
 		)
